File: DeluxeFloppy.sch (KiCad schematic (older format))
At the start: 48 parts, among them P1 Floppy, P2 Serial Port, SW1 Serial Port Config, SW2 Boot ROM Address, SW3 Enable ROM, SW4 ROM Write-Protect, SW5 28C64B Mode, U1 82077AA/PC8477, U2 16(C)x50, U3 GD75232, U4 Boot ROM, U5 74LS688, U6 74LS138, U7 74LS138, U8 1.8432MHz TTL, X1 24MHz, X2 1.8432MHz

Commit message: Add files via upload
Parts:
- removed BUS1: BUSPC_DEV, Custom:Conn_Bus_ISA8, symbol isa_fdc-monotech-modified-rescue:BUSPC_DEV
- removed HOLE1, HOLE2: CONN_1, MountingHole:MountingHole_3.2mm_M3_Pad, symbol isa_fdc-monotech-modified-rescue:CONN_1
- removed JP2: D7_Pulldown, Jumper:SolderJumper-2_P1.3mm_Open_RoundedPad1.0x1.5mm, symbol Jumper:SolderJumper_2_Open
- removed JP3: Enable Floppy, Jumper:SolderJumper-2_P1.3mm_Open_RoundedPad1.0x1.5mm, symbol Jumper:SolderJumper_2_Open
- removed P2: Serial Port, Custom:Conn_Dsub_DE9M, symbol isa_fdc-monotech-modified-rescue:DB9
- removed R1, R2: 10K, Resistor_THT:R_Axial_DIN0207_L6.3mm_D2.5mm_P7.62mm_Horizontal, symbol Device:R
- removed RN1: 10K, Resistor_THT:R_Array_SIP8, symbol Device:R_Network07
- removed RN2: 1K, Resistor_THT:R_Array_SIP8, symbol Device:R_Network07
- removed SW2: Boot ROM Address, Button_Switch_THT:SW_DIP_SPSTx04_Slide_9.78x12.34mm_W7.62mm_P2.54mm, symbol Switch:SW_DIP_x04
- removed SW3: Enable ROM, Button_Switch_THT:SW_CuK_OS102011MA1QN1_SPDT_Angled, symbol Switch:SW_SPDT
- removed SW4: ROM Write-Protect, Button_Switch_THT:SW_CuK_OS102011MA1QN1_SPDT_Angled, symbol Switch:SW_SPDT
- removed SW5: 28C64B Mode, Custom:SW_MS-22D18G2, symbol Switch:SW_DPDT_x2
- removed U3: GD75232, Package_SO:SSOP-20_5.3x7.2mm_P0.65mm, symbol isa_fdc-monotech-modified-rescue:GD75232
- removed U5: 74LS688, Package_DIP:DIP-20_W7.62mm, symbol isa_fdc-monotech-modified-rescue:74LS688
- removed U6, U7: 74LS138, Package_DIP:DIP-16_W7.62mm, symbol isa_fdc-monotech-modified-rescue:74LS138
- removed U8: 1.8432MHz TTL, Oscillator:Oscillator_DIP-14, symbol isa_fdc-monotech-modified-rescue:OSC
- added BUS1: Bus_ISA_8bit, Custom:Conn_Bus_ISA8, symbol Connector:Bus_ISA_8bit
- added C20: 104, Capacitor_SMD:C_0805_2012Metric, symbol isa_fdc-monotech-modified-rescue:C
- added JP1: FDC_En, Jumper:SolderJumper-2_P1.3mm_Bridged_Pad1.0x1.5mm, symbol Jumper:SolderJumper_2_Bridged
- added LOGO1: SYM_Arrow45_Large, Custom KiCad Library:Monotech Logo 14mm, symbol Graphic:SYM_Arrow45_Large
- added LOGO2: SYM_Arrow45_Large, Custom:DeluxeFloppy, symbol Graphic:SYM_Arrow45_Large
- added NT1: Net-Tie_2, NetTie:NetTie-2_SMD_Pad0.5mm, symbol Device:Net-Tie_2
- added P1: Serial Port, Custom KiCad Library:Conn_Dsub_DE9M, symbol Connector:DB9_Male
- added P3: Floppy, Custom:Connector_Edge_FloppyDisk, symbol isa_fdc-monotech-modified-rescue:CONN_17X2
- added RN1, RN4, RN5: 10k, Resistor_SMD:R_Array_Convex_4x0603, symbol Device:R_Pack04
- added RN2, RN3: 1k, Resistor_SMD:R_Array_Convex_4x0603, symbol Device:R_Pack04
- added SW2: ROM Config, Button_Switch_THT:SW_DIP_SPSTx08_Slide_9.78x22.5mm_W7.62mm_P2.54mm, symbol Switch:SW_DIP_x08
- added U1, U7: AHCT138, Custom KiCad Library:SOIC-16_3.9x9.9mm_P1.27mm, symbol 74xx:74LS138
- added U2: HCT245, Custom KiCad Library:SOIC-20W_7.5x12.8mm_P1.27mm, symbol 74xx:74LS245
- added U3: HCT00, Custom KiCad Library:SOIC-14_3.9x8.7mm_P1.27mm, symbol 74xx:74LS00
- added U5: GD75232, Custom KiCad Library:TSSOP-20_4.4x6.5mm_P0.65mm, symbol Interface_UART:GD75232PW
- added U6: HCT86, Custom KiCad Library:SOIC-14_3.9x8.7mm_P1.27mm, symbol 74xx:74LS86
- added U8: AHCT1G02, Package_SO:TSOP-5_1.65x3.05mm_P0.95mm, symbol 74xGxx:74AHC1G02
- C1: renamed from C18; value 22pF -> 22; footprint Capacitor_THT:C_Disc_D4.3mm_W1.9mm_P5.00mm -> Capacitor_SMD:C_0805_2012Metric
- C10: renamed from C5; value 0.1uF -> 104; footprint Capacitor_THT:C_Disc_D4.3mm_W1.9mm_P5.00mm -> Capacitor_SMD:C_0805_2012Metric
- C11: renamed from C6; value 0.1uF -> 104; footprint Capacitor_THT:C_Disc_D4.3mm_W1.9mm_P5.00mm -> Capacitor_SMD:C_0805_2012Metric
- C12: renamed from C7; value 0.1uF -> 104; footprint Capacitor_THT:C_Disc_D4.3mm_W1.9mm_P5.00mm -> Capacitor_SMD:C_0805_2012Metric
- C13: renamed from C8; value 0.1uF -> 104; footprint Capacitor_THT:C_Disc_D4.3mm_W1.9mm_P5.00mm -> Capacitor_SMD:C_0805_2012Metric
- C14: renamed from C11; value 10uF -> 106; footprint Capacitor_THT:C_Disc_D4.3mm_W1.9mm_P5.00mm -> Capacitor_SMD:C_0805_2012Metric
- C15: renamed from C12; value 10uF -> 106; footprint Capacitor_THT:C_Disc_D4.3mm_W1.9mm_P5.00mm -> Capacitor_SMD:C_0805_2012Metric
- C16: renamed from C9; value 0.1uF -> 104; footprint Capacitor_THT:C_Disc_D4.3mm_W1.9mm_P5.00mm -> Capacitor_SMD:C_0805_2012Metric
- C17: renamed from C13; value 10uF -> 106; footprint Capacitor_THT:C_Disc_D4.3mm_W1.9mm_P5.00mm -> Capacitor_SMD:C_0805_2012Metric
- C18: renamed from C10; value 0.1uF -> 104; footprint Capacitor_THT:C_Disc_D4.3mm_W1.9mm_P5.00mm -> Capacitor_SMD:C_0805_2012Metric
- C19: renamed from C14; value 10uF -> 106; footprint Capacitor_THT:C_Disc_D4.3mm_W1.9mm_P5.00mm -> Capacitor_SMD:C_0805_2012Metric
- C2: renamed from C19; value 47pF -> 47; footprint Capacitor_THT:C_Disc_D4.3mm_W1.9mm_P5.00mm -> Capacitor_SMD:C_0805_2012Metric
- C3: renamed from C15; value 22pF -> 22; footprint Capacitor_THT:C_Disc_D4.3mm_W1.9mm_P5.00mm -> Capacitor_SMD:C_0805_2012Metric
- C4: renamed from C16; value 22pF -> 22; footprint Capacitor_THT:C_Disc_D4.3mm_W1.9mm_P5.00mm -> Capacitor_SMD:C_0805_2012Metric
- C5: renamed from C17; value 4.7nF -> 473; footprint Capacitor_THT:C_Disc_D4.3mm_W1.9mm_P5.00mm -> Capacitor_SMD:C_0805_2012Metric
- C6: renamed from C1; value 0.1uF -> 104; footprint Capacitor_THT:C_Disc_D4.3mm_W1.9mm_P5.00mm -> Capacitor_SMD:C_0805_2012Metric
- C7: renamed from C2; value 0.1uF -> 104; footprint Capacitor_THT:C_Disc_D4.3mm_W1.9mm_P5.00mm -> Capacitor_SMD:C_0805_2012Metric
- C8: renamed from C3; value 0.1uF -> 104; footprint Capacitor_THT:C_Disc_D4.3mm_W1.9mm_P5.00mm -> Capacitor_SMD:C_0805_2012Metric
- C9: renamed from C4; value 0.1uF -> 104; footprint Capacitor_THT:C_Disc_D4.3mm_W1.9mm_P5.00mm -> Capacitor_SMD:C_0805_2012Metric
- P2: renamed from P1; footprint Custom:Pin_Header_Straight_2x17_Pitch2.54mm_shrouded -> Connector_IDC:IDC-Header_2x17_P2.54mm_Vertical
- R1: renamed from R3; footprint Resistor_THT:R_Axial_DIN0207_L6.3mm_D2.5mm_P7.62mm_Horizontal -> Resistor_SMD:R_0805_2012Metric
- R2: renamed from R4; footprint Resistor_THT:R_Axial_DIN0207_L6.3mm_D2.5mm_P7.62mm_Horizontal -> Resistor_SMD:R_0805_2012Metric
- SW1: value Serial Port Config -> UART Config
- U4: renamed from U2; value 16(C)x50 -> 16C550_QFP; footprint Package_LCC:PLCC-44_THT-Socket -> Package_QFP:LQFP-48_7x7mm_P0.5mm; symbol isa_fdc-monotech-modified-rescue:16550-PLCC -> 16550-lqfp:16550-LQFP
- U9: renamed from U4; value Boot ROM -> 28C256; footprint Package_DIP:DIP-28_W15.24mm_Socket -> Custom KiCad Library:DIP-28_W15.24mm_Socket
- X1: renamed from X2; footprint Crystal:Crystal_HC49-U_Horizontal_1EP_style2 -> Crystal:Crystal_HC49-U_Horizontal_1EP_style1; symbol isa_fdc-monotech-modified-rescue:CRYSTAL -> Device:Crystal_GND3
- X2: renamed from X1; footprint Crystal:Crystal_HC49-4H_Vertical -> Crystal:Crystal_SMD_5032-2Pin_5.0x3.2mm
- renumbered JP1 to JP2, U1 to U10
Connections:
- net -12V: now also BUS1.7 (-12V), U5.10 (VSS)
- net 0x2E8: now also U1.11 (O4)
- net 0x2F8: now also U1.9 (O6)
- net 0x3E8: now also U1.10 (O5)
- net 0x3F0: now also JP1.1 (A), U1.12 (O3)
- net 0x3F8: now also U1.7 (O7)
- net 12V: now also BUS1.9 (+12V), U5.1 (VDD)
- net A0: now also U4.28 (A0), BUS1.62 (BA00); no longer U4.31 (A0)
- net A1: now also U4.27 (A1), BUS1.61 (BA01); no longer U4.30 (A1)
- net A10: now also BUS1.52 (BA10)
- net A11: now also BUS1.51 (BA11)
- net A12: now also BUS1.50 (BA12)
- net A13: now also BUS1.49 (BA13), SW2.6
- net A14: now also BUS1.48 (BA14), SW2.5
- net A15: now also BUS1.47 (BA15), U6.5
- net A16: now also BUS1.46 (BA16), U6.2
- net A17: now also BUS1.45 (BA17), U8.2
- net A18: now also BUS1.44 (BA18), U3.12
- net A19: now also BUS1.43 (BA19), U3.13
- net A2: now also U4.26 (A2), BUS1.60 (BA02); no longer U4.29 (A2)
- net A3: now also BUS1.59 (BA03), U1.3 (A2)
- net A4: now also BUS1.58 (BA04), U1.2 (A1)
- net A5: now also BUS1.57 (BA05), U3.4
- net A6: now also BUS1.56 (BA06), U3.5
- net A7: now also BUS1.55 (BA07), U3.1
- net A8: now also BUS1.54 (BA08), U1.1 (A0)
- net A9: now also BUS1.53 (BA09), U3.2
- net AEN: now also BUS1.42 (AEN), SW2.7, U3.10
- net CTS: now also P1.8, U5.7 (RA4)
- net D0: now also BUS1.40 (DB0), U2.2 (A0); no longer U4.2 (D0)
- net D1: now also BUS1.39 (DB1), U2.3 (A1); no longer U4.3 (D1)
- net D2: now also BUS1.38 (DB2), U2.4 (A2); no longer U4.4 (D2)
- net D3: now also BUS1.37 (DB3), U2.5 (A3); no longer U4.5 (D3)
- net D4: now also BUS1.36 (DB4), U2.6 (A4); no longer U4.6 (D4)
- net D5: now also BUS1.35 (DB5), U2.7 (A5); no longer U4.7 (D5)
- net D6: now also BUS1.34 (DB6), U2.8 (A6); no longer U4.8 (D6)
- net D7: now also BUS1.33 (DB7), U2.9 (A7); no longer U4.9 (D7)
- net DCD: now also P1.1, U5.2 (RA1)
- net DENSL: now also P3.2 (P2)
- net DIR: now also P3.18 (P18)
- net DRQ2: now also BUS1.6 (DRQ2)
- net DSA: now also P3.14 (P14)
- net DSB: now also P3.12 (P12)
- net DSKCG: now also P3.34 (P34), RN3.1 (R1.1)
- net DSR: now also P1.6, U5.3 (RA2)
- net DTR: now also P1.4, U5.8 (DY3)
- net GND: now also U4.17 (WR), U4.18 (GND), U4.20 (RD), U4.24 (~ADS), X1.3, BUS1.1 (GND), BUS1.10 (GND), BUS1.31 (GND), C20.2, NT1.1, P3.1 (P1), P3.11 (P11), P3.13 (P13), P3.15 (P15), P3.19 (P19), P3.21 (P21), P3.23 (P23), P3.25, P3.29 (P29), P3.31 (P31), P3.5 (P5), P3.7 (P7), RN4.3 (R3.1), RN4.4 (R4.1), RN5.1 (R1.1), RN5.2 (R2.1), RN5.3 (R3.1), RN5.4 (R4.1), U1.8 (GND), U2.10 (GND), U3.7 (GND), U5.11 (GND), U6.7 (GND), U7.8 (GND), U8.3 (GND); no longer U4.21 (WR), U4.22 (GND), U4.25 (RD), U4.28 (~ADS)
- net HDSEL: now also P3.32 (P32)
- net INDEX: now also P3.8 (P8), RN2.1 (R1.1)
- net IRQ3: now also BUS1.25 (IRQ3)
- net IRQ4: now also BUS1.24 (IRQ4)
- net IRQ5: now also BUS1.23 (IRQ5)
- net IRQ6: now also BUS1.22 (IRQ6)
- net IRQ7: now also BUS1.21 (IRQ7)
- net MEA: now also P3.10 (P10)
- net MEB: now also P3.16 (P16)
- net RDATA: now also P3.30 (P30), RN2.4 (R4.1)
- net RI: now also P1.9, U5.9 (RA5)
- net RSTDRV: now also U4.35 (MR), BUS1.2 (RESET); no longer U4.39 (MR)
- net RTS: now also P1.7, U5.5 (DY1)
- net RX: now also P1.2, U5.4 (RA3)
- net SIN: now also U4.7 (SIN), U5.17 (RY3); no longer U4.11 (SIN)
- net SOUT: now also U4.8 (SOUT), U5.15 (DA2); no longer U4.13 (SOUT)
- net STEP: now also P3.20 (P20)
- net TC: now also BUS1.27 (TC)
- net TRK00: now also P3.26 (P26), RN2.2 (R2.1)
- net TX: now also P1.3, U5.6 (DY2)
- net UART_IRQ: now also U4.30 (INTR); no longer U4.33 (INTR)
- net VCC: now also U4.10 (CS1), U4.42 (VCC), U4.9 (CS0), BUS1.29 (VCC), BUS1.3 (VCC), C20.1, RN1.3 (R3.1), RN1.4 (R4.1), RN2.5 (R4.2), RN2.6 (R3.2), RN2.7 (R2.2), RN2.8 (R1.2), RN3.8 (R1.2), RN4.1 (R1.1), RN4.2 (R2.1), SW2.1, SW2.2, SW2.3, SW2.4, U1.16 (VCC), U2.20 (VCC), U3.14 (VCC), U3.9, U5.20 (VCC), U6.14 (VCC), U7.16 (VCC), U8.5 (VCC); no longer U4.14 (CS0), U4.15 (CS1), U4.44 (VCC)
- net WDATA: now also P3.22 (P22)
- net WE: now also P3.24 (P24)
- net WP: now also P3.28 (P28), RN2.3 (R3.1)
- net ~CTS: now also U4.38 (~CTS), U5.14 (RY4); no longer U4.40 (~CTS)
- net ~DACK2: now also BUS1.26 (~DACK2)
- net ~DCD: now also U4.40 (~DCD), U5.19 (RY1); no longer U4.42 (~DCD)
- net ~DSR: now also U4.39 (~DSR), U5.18 (RY2); no longer U4.41 (~DSR)
- net ~DTR: now also U4.33 (~DTR), U5.13 (DA3); no longer U4.37 (~DTR)
- net ~IOR: now also U4.19 (~RD), BUS1.14 (~IOR), U2.1 (A->B); no longer U4.24 (~RD)
- net ~IOW: now also U4.16 (~WR), BUS1.13 (~IOW); no longer U4.20 (~WR)
- net ~MEMR: now also BUS1.12 (~SMEMR)
- net ~MEMW: now also BUS1.11 (~SMEMW), SW2.8
- net ~RI: now also U4.41 (~RI), U5.12 (RY5); no longer U4.43 (~RI)
- net ~ROMW: now also RN4.8 (R1.2), SW2.9
- net ~ROM_CS: now also U7.15 (O0)
- net ~RTS: now also U4.32 (~RTS), U5.16 (DA1); no longer U4.36 (~RTS)
- net ~UART_CS: now also U4.11 (~CS2), RN1.5 (R4.2), U2.19 (CE); no longer U4.16 (~CS2)
- net at C1.2, R2.1, X1.1: now also U4.14 (XIN); no longer U4.18 (XIN)
- net DRATE0: now reaches P2.6 (P6), U10.28 (DRATE0)
- net DRATE0: now also P3.6 (P6)
- net ~FDC_CS: now reaches U10.6 (CS)
- net ~FDC_CS: now also JP1.2 (B), RN1.6 (R3.2)
- net at U4.12 (~BAUDOUT): now also U4.5 (RCLK)
- net at R1.2: now also U4.15 (XOUT); no longer U4.19 (XOUT)
- new net: U1.4 (E1), U3.3
- new net: U1.5 (E2), U3.6
- new net: U1.6 (E3), U3.8
- new net: RN4.5 (R4.2), SW2.12, U6.10
- new net: RN4.6 (R3.2), SW2.11, U6.13
- new net: RN4.7 (R2.2), SW2.10, U8.1
- new net: RN5.5 (R4.2), SW2.16, U6.1
- new net: U6.3, U7.1 (A0)
- new net: RN5.6 (R3.2), SW2.15, U6.4
- new net: U6.6, U7.2 (A1)
- new net: U6.8, U7.3 (A2)
- new net: RN5.7 (R2.2), SW2.14, U6.9
- new net: U6.11, U7.5 (E2)
- new net: RN5.8 (R1.2), SW2.13, U6.12
- new net: U3.11, U7.4 (E1)
- new net: U7.6 (E3), U8.4
- new net: NT1.2, P1.5
- new net DB0: U2.18 (B0), U4.43 (D0)
- new net DB1: U2.17 (B1), U4.44 (D1)
- new net DB2: U2.16 (B2), U4.45 (D2)
- new net DB3: U2.15 (B3), U4.46 (D3)
- new net DB4: U2.14 (B4), U4.47 (D4)
- new net DB5: U2.13 (B5), U4.2 (D5)
- new net DB6: U2.12 (B6), U4.3 (D6)
- new net DB7: U2.11 (B7), U4.4 (D7)
- no-connect marks 44 -> 55
Other:
- note added: "5.25" edge connector"
- note added: "ROM Address:\n1234 ROM\n0000 C0000*\n0001 C2000\n0010 C4000\n0011 C6000\n0100 C8000*\n0101 CA000\n0110 CC000\n0111 CE000\n1000 D0000* !\n1001 D2000\n1010 D4000\n1011 D6000\n1100 D8000*\n1101 DA000\n1110 DC000\n1111 DE000"
- note added: "Serial Port IRQ: SW1-4\nSerial Port I/O Address: SW5-8\n\n1: IRQ3 (COM2/4)\n2: IRQ4 (COM1/3)\n3: IRQ5\n4: IRQ7\n\n5: 2E8 (COM4)\n6: 3E8 (COM3)\n7: 2F8 (COM2)\n8: 3F8 (COM1)\n\n! = Default\n* = 32K ROM support\n\nROM Size:\n5/6 ON - 8K: 27(C)64, 28C64B\n5/6 OFF - 32K: 28C256\n\n7: ROM Enable\n8: ROM Write Enable"
- note removed: "Mount Holes"
- note removed: "Optional crystal circuit\ninstead of oscillator"
- note removed: "SW1.1 - ON: Use IRQ3 for UART (COM2, COM4)\nSW1.2 - ON: Use IRQ4 for UART (COM1, COM3)\nSW1.3 - ON: Use IRQ5 for UART\nSW1.4 - ON: Use IRQ7 for UART\nSW1.5 - ON: Set UART address to 0x2E8 (COM4)\nSW1.6 - ON: Set UART address to 0x3E8 (COM3)\nSW1.7 - ON: Set UART address to 0x2F8 (COM2)\nSW1.8 - ON: Set UART address to 0x3F8 (COM1)\n\nSW2.1 - ON: ROM A16 = 0; OFF: ROM A16 = 1\nSW2.2 - ON: ROM A15 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"
- moved on the sheet: C1, C10, C11, C12, C13, C14, C15, C2, C6, C7, C8, C9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
